File: tinywhoop_frame/tinywhoop_frame-backups/tinywhoop_frame-2025-12-08_000207/_autosave-tinywhoop_frame.kicad_pcb (KiCad board)
At the start: 2 copper layers, 90 x 90 mm, 17 parts, among them J1 ESP_conn1, J2 ESP_conn2, J3 ESP_Unused_Pins1, J5 Batt_conn, J6 Conn_02x03_Counter_Clockwise, Q1 2N7002, Q2 2N7002, Q3 2N7002, Q4 2N7002

Commit message: pcb updates, created fab files
Parts:
- removed J6: Conn_02x03_Counter_Clockwise, Connector_PinSocket_2.54mm:PinSocket_2x03_P2.54mm_Vertical
- added J4: Conn_02x03_Counter_Clockwise, Connector_PinHeader_2.54mm:PinHeader_2x03_P2.54mm_Vertical, F.Cu at (162.0, 65.5)
Connections:
- J2 pad 4: /GPIO9 -> Net-(J2-Pin_4)
- J2 pad 5: /GPIO8 -> Net-(J2-Pin_5)
- J2 pad 6: /GPIO7 -> Net-(J2-Pin_6)
- J2 pad 7: /GPIO44 -> Net-(J2-Pin_7)
Routing:
- net /GPIO44: track 11.9 -> 0.00 mm
- net Net-(J2-Pin_7): track 0.00 -> 11.9 mm
- net /GPIO7: track 8.31 -> 0.00 mm
- net Net-(J2-Pin_6): track 0.00 -> 8.29 mm
- net /GPIO9: track 4.72 -> 0.00 mm
- net /GPIO8: track 4.72 -> 0.00 mm
- net Net-(J2-Pin_5): track 0.00 -> 4.70 mm
- net Net-(J2-Pin_4): track 0.00 -> 4.70 mm
