File: tinywhoop_frame/tinywhoop_frame.kicad_pcb (KiCad board)
At the start: 2 copper layers, 70 x 70 mm, 27 parts, among them J1 ESP_conn1, J2 ESP_conn2, J3 ESP_Unused_Pins1, J4 Batt_conn_MCU, J5 Batt_conn_LIPO, J6 Conn_02x03_Counter_Clockwise, Q1 2N7002, Q2 2N7002, Q3 2N7002, Q4 2N7002

Commit message: pcb update
Connections:
- J6 pad 1: unconnected-(J6-Pin_1-Pad1) -> BATT-
Other:
- board text added: "+"
- board text added: "3V3"
- board text added: "7"
- board text added: "8"
- board text added: "9"
- board text added: "GND"
- board text added: "M1+"
- board text added: "M1-"
- board text added: "M2+"
- board text added: "M2-"
- board text added: "M3+"
- board text added: "M3-"
- board text added: "M4+"
- board text added: "M4-"
- board text added: "RX"
- board text added: "SCL"
- board text added: "SDA"
- board text added: "TX"
